Commit message: could controll through CLI

File: ros_gui/urdf/default.xacro (robot description, xacro)
@@ -362,7 +362,45 @@
 		<axis xyz="0 0 1" />
 	</joint>
+	<!-- ===================================================== -->
+	<!-- transmission elements -->
+<transmission name="front_right_motor_joint" >
+		<type>transmission_interface/SimpleTransmission</type>
+		<joint name="joint_front_right_prop">
+			<hardwareInterface>hardware_interface/EffortJointInterface</hardwareInterface>
+		</joint>
+		<actuator name="BLDC_motor1">
+			<mechanicalReduction>1</mechanicalReduction>
+		</actuator>
+	</transmission>
+	<transmission name="front_left_motor_joint" >
+		<type>transmission_interface/SimpleTransmission</type>
+		<joint name="joint_front_left_prop">
+			<hardwareInterface>hardware_interface/EffortJointInterface</hardwareInterface>
+		</joint>
+		<actuator name="BLDC_motor2">
+			<mechanicalReduction>1</mechanicalReduction>
+		</actuator>
+	</transmission>
+	<transmission name="back_right_motor_joint" >
+		<type>transmission_interface/SimpleTransmission</type>
+		<joint name="joint_back_right_prop">
+			<hardwareInterface>hardware_interface/EffortJointInterface</hardwareInterface>
+		</joint>
+		<actuator name="BLDC_motor3">
+			<mechanicalReduction>1</mechanicalReduction>
+		</actuator>
+	</transmission>
+	<transmission name="back_left_motor_joint" >
+		<type>transmission_interface/SimpleTransmission</type>
+		<joint name="joint_back_left_prop">
+			<hardwareInterface>hardware_interface/EffortJointInterface</hardwareInterface>
+		</joint>
+		<actuator name="BLDC_motor4">
+			<mechanicalReduction>1</mechanicalReduction>
+		</actuator>
+	</transmission>
 <!-- ======================================================== -->
 <!-- Add transmission elements -->
-	<transmission name="front_right_motor_joint" >
+	<!-- <transmission name="front_right_motor_joint" >
 		<type>transmission_interface/SimpleTransmission</type>
 		<joint name="joint_front_right_prop">
@@ -403,4 +441,4 @@
 			<mechanicalReduction>1</mechanicalReduction>
 		</actuator>
-	</transmission>
+	</transmission> -->
 </robot>
